File: pcb/windpup/windpup.kicad_pcb (KiCad board)
At the start: 2 copper layers, 50.3 x 46.2 mm, 33 parts, among them J1 USB_C_Receptacle_USB2.0, J2 Conn_ARM_JTAG_SWD_10, J3 DB25_Female, SW1 push, U1 MAX3237, U2 TLV1117-33, U3 ESP-C3-WROOM-02, U4 TLC59211

Commit message: pcb: update for manuf
Parts:
- added C1: 22p, Capacitor_SMD:C_0805_2012Metric_Pad1.18x1.45mm_HandSolder, B.Cu at (148.5, 102.3)
- added C14: 0.1u, Capacitor_SMD:C_0805_2012Metric_Pad1.18x1.45mm_HandSolder, F.Cu at (151.6, 108.5)
- added C2: 22p, Capacitor_SMD:C_0805_2012Metric_Pad1.18x1.45mm_HandSolder, B.Cu at (151.6, 102.4)
- added D9: ESD9B5.0ST5G, Diode_SMD:D_SOD-923, F.Cu at (153.9, 113.3)
- added SW2: SW_SPDT, feet:NidecCopal_CL-SB-12B-xx, F.Cu at (145.3, 110.6)
- added U5: TPD2E2U06, Package_TO_SOT_SMD:SOT-563, F.Cu at (150.0, 99.3)
- JP1: footprint Jumper:SolderJumper-2_P1.3mm_Bridged_RoundedPad1.0x1.5mm -> Jumper:SolderJumper-2_P1.3mm_Open_RoundedPad1.0x1.5mm
- moved R1 13.7 mm to (143.3, 118.1), turned to 90 degrees
- moved R2 13.7 mm to (157.0, 118.1), turned to 90 degrees
- moved JP1 0.59 mm to (151.8, 92.6)
- moved C10 0.25 mm to (158.0, 81.0)
Connections:
- R1 pad 1: Net-(J1-PadB5) -> GND
- R1 pad 2: GND -> Net-(J1-PadA5)
- R2 pad 1: Net-(J1-PadA5) -> GND
- R2 pad 2: GND -> Net-(J1-PadB5)
- RN1 pad 10: GND -> +3V3
- RN1 pad 11: GND -> +3V3
- RN1 pad 12: GND -> +3V3
- RN1 pad 13: GND -> +3V3
- RN1 pad 14: GND -> +3V3
- RN1 pad 15: GND -> +3V3
- RN1 pad 16: GND -> +3V3
- RN1 pad 9: GND -> +3V3
- U3 pad 8: (no net) -> /BOOTMODE
Routing:
- net +3V3: track 105.1 -> 119.3 mm
- net /BOOTMODE: track 0.00 -> 4.69 mm
- net /D+: track 37.3 -> 41.2 mm, vias 1 -> 2
- net /D-: track 37.3 -> 41.2 mm, vias 1 -> 2
- net /EN: track 27.6 -> 30.3 mm
- net VBUS: track 17.4 -> 20.0 mm
- net ESP_CTS: track 20.4 -> 22.0 mm
- net RS232_RTS: track 20.1 -> 21.6 mm
- net RS232_TxD: track 25.8 -> 26.9 mm
- net RS232_RxD: track 26.1 -> 27.1 mm
- net RS232_DCE_RDY: track 15.8 -> 16.8 mm
- net ESP_TxD: track 23.4 -> 24.3 mm
- net RS232_CTS: track 22.3 -> 22.8 mm
- net GND: vias 15 -> 17
Other:
- outline, holes or cut-outs redrawn
- board text added: "JLCJLCJLCJLC"
- board text added: "coffeeware 4 zoomies"
- board text added: "erin moon 2021"
- board text added: "funny lightbulb goes here"
- board text added: "windpup"
- board text removed: "JLCJLCJLC"
