File: pcb/windpup/windpup.sch (KiCad schematic (older format))
At the start: 35 parts, among them J1 USB_C_Receptacle_USB2.0, J2 Conn_ARM_JTAG_SWD_10, J3 DB25_Female, SW1 push, U1 MAX3237, U2 TLV1117-33, U3 ESP-C3-WROOM-02, U4 TLC59211

Commit message: pcb: update for manuf
Parts:
- removed R1, R2: 5.1k, Resistor_SMD:R_0805_2012Metric_Pad1.20x1.40mm_HandSolder, symbol Device:R
- added C14: 0.1u, Capacitor_SMD:C_0805_2012Metric_Pad1.18x1.45mm_HandSolder, symbol Device:C
- added D9: ESD9B5.0ST5G, Diode_SMD:D_SOD-923, symbol Diode:ESD9B5.0ST5G
- added R1, R2: 5.1k, Resistor_SMD:R_0805_2012Metric_Pad1.20x1.40mm_HandSolder, symbol Device:R_Small
- added SW2: SW_SPDT, feet:NidecCopal_CL-SB-12B-xx, symbol Switch:SW_SPDT
- added U5: TPD2E2U06, Package_TO_SOT_SMD:SOT-563, symbol Power_Protection:TPD2E2U06
- C1, C2: footprint (none) -> Capacitor_SMD:C_0805_2012Metric_Pad1.18x1.45mm_HandSolder; dkpn (none) -> 1276-2606-1-ND
- C10, C11, C12: dkpn (none) -> 1276-6470-1-ND
- C9: dkpn (none) -> 1276-6478-1-ND
- D1, D2, D3, D4, D5, D6, D7, D8: dkpn (none) -> 754-1116-1-ND
- J2: dkpn (none) -> S9012E-05-ND
- J3: dkpn (none) -> 2057-DB25-ST-1-ND
- JP1: footprint Jumper:SolderJumper-2_P1.3mm_Bridged_RoundedPad1.0x1.5mm -> Jumper:SolderJumper-2_P1.3mm_Open_RoundedPad1.0x1.5mm
- R3: dkpn (none) -> 311-10.0KCRCT-ND
- R4: dkpn (none) -> 311-1.00KCRCT-ND
- RN1: dkpn (none) -> CAT16-221J8LFCT-ND
- SW1: dkpn (none) -> CKN10284CT-ND
- U1: dkpn (none) -> 296-19801-1-ND
- U2: dkpn (none) -> 296-31967-1-ND
- U4: dkpn (none) -> 296-25404-1-ND
Connections:
- net +3V3: now also RN1.10 (R7.2), RN1.11 (R6.2), RN1.12 (R5.2), RN1.13 (R4.2), RN1.14 (R3.2), RN1.15 (R2.2), RN1.16 (R1.2), RN1.9 (R8.2)
- net D+: now also U5.5
- net D-: now also U5.3
- net GND: now also C14.2, D9.2 (A2), R1.1, R2.1, SW2.2 (B), U5.4; no longer RN1.10 (R7.2), RN1.11 (R6.2), RN1.12 (R5.2), RN1.13 (R4.2), RN1.14 (R3.2), RN1.15 (R2.2), RN1.16 (R1.2), RN1.9 (R8.2)
- net VBUS: now also C14.1, D9.1 (A1)
- net BOOTMODE: now reaches U3.8 (IO9)
- net BOOTMODE: now also SW2.3 (C)
- net at J1.A5 (CC1): now also R1.2
- net at J1.B5 (CC2): now also R2.2
- no-connect marks 5 -> 27
Other:
- note added: "TODO validate IO2"
- note added: "VALID"
- note added: "pinout valid\nsemantics ??"
- note added: "todo: should this be inverted?"
- note removed: "TODO prot diodes"
- moved on the sheet: J2
